File: DMH_VCF_Diode_Ladder_PCB/Inputs_and_Outputs.kicad_sch (KiCad schematic)
At the start: 0 parts

Commit message: Finished schematic and added Bus CV 2 pot
Parts:
- added J1, J2, J3, J4, J5: TS_Jack_6.35mm_Sw, SynthStuff:CUI_MJ-63052A, symbol SynthStuff:TS_Jack_6.35mm_Sw
- added J200: IDC_02x05, SynthStuff:IDC-Header_2x05_P2.54mm_Vertical_BackBone, symbol SynthStuff:BackBone_Connector_10Pin
- added J50: Conn_01x06, symbol Connector_Generic:Conn_01x06
- added J60: Conn_01x06, Connector_PinSocket_2.54mm:PinSocket_1x06_P2.54mm_Vertical, symbol Connector_Generic:Conn_01x06
Connections:
- new net: J1.TN, J200.1 (Pin_1), J60.1 (Pin_1)
- new net: J2.TN, J200.2 (Pin_2), J60.2 (Pin_2)
- new net: J200.6 (Pin_6), J4.TN, J60.4 (Pin_4)
- new net: J200.7 (Pin_7), J5.TN, J60.5 (Pin_5)
- new net Bus CV In: J3.TN, J60.3 (Pin_3)
- new net CV 1 Jack: J2.T, J50.2 (Pin_2)
- new net CV 2 Jack: J3.T, J50.3 (Pin_3)
- new net CV 3 Jack: J4.T, J50.4 (Pin_4)
- new net GND: J1.S, J2.S, J200.10 (Pin_10), J200.3 (Pin_3), J200.4 (Pin_4), J200.5 (Pin_5), J200.8 (Pin_8), J200.9 (Pin_9), J3.S, J4.S, J5.S, J50.6 (Pin_6), J60.6 (Pin_6)
- new net Input Jack: J1.T, J50.1 (Pin_1)
- new net Output Jack: J5.T, J50.5 (Pin_5)

Commit message: Added Bus CV On Off switch
Parts:
- added SW4: SW_SPDT_321_OnOff, SynthStuff:Toggle_Switch_THT, symbol SynthStuff:SW_SPDT_321_OnOff
Connections:
- net Bus CV In: now also SW4.2 (B); no longer J3.TN, J60.3 (Pin_3)
- new net: J3.TN, J60.3 (Pin_3), SW4.1 (C)
- no-connect marks 0 -> 1
Other:
- note added: "Connectors PCB"
Changed lines of the file:
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@@
 		(color 0 0 0 0)
 	)
+	(no_connect
+		(at 176.53 62.23)
+	)
+	(wire
+		(pts
+			(xy 142.24 57.15) (xy 176.53 57.15)
+		)
+		(stroke
+			(width 0)
+			(type default)
+		)
+	)
 	(wire
 		(pts
@@
 	(wire
 		(pts
+			(xy 186.69 59.69) (xy 194.31 59.69)
+		)
+		(stroke
+			(width 0)
+			(type default)
+		)
+	)
+	(wire
+		(pts
 			(xy 139.7 59.69) (xy 139.7 48.26)
 		)
@@
 	(wire
 		(pts
-			(xy 142.24 57.15) (xy 177.8 57.15)
-		)
-		(stroke
-			(width 0)
-			(type default)
-		)
-	)
-	(wire
-		(pts
 			(xy 132.08 48.26) (xy 139.7 48.26)
 		)
@@
 			(width 0)
 			(type default)
+		)
+	)
+	(rectangle
+		(start 25.4 25.4)
+		(end 119.38 152.4)
+		(stroke
+			(width 0)
+			(type default)
+		)
+		(fill
+			(type none)
+		)
+	)
+	(text "Connectors PCB"
+		(exclude_from_sim no)
+		(at 110.998 151.13 0)
+		(effects
+			(font
+				(size 1.27 1.27)
+			)
 		)
 	)
@@
 	(hierarchical_label "Bus CV In"
 		(shape input)
-		(at 177.8 57.15 0)
+		(at 194.31 59.69 0)
 		(fields_autoplaced yes)
 		(effects
@@
 					(unit 1)
 				)
+			)
+		)
+	)
+	(symbol
+		(lib_id "SynthStuff:SW_SPDT_321_OnOff")
+		(at 181.61 59.69 180)
+		(unit 1)
+		(exclude_from_sim no)
+		(in_bom yes)
+		(on_board yes)
+		(dnp no)
+		(fields_autoplaced yes)
+		(property "Reference" "SW4"
+			(at 181.61 50.8 0)
+			(effects
+				(font
+					(size 1.27 1.27)
+				)
+			)
+		)
+		(property "Value" "SW_SPDT_321_OnOff"
+			(at 181.61 53.34 0)
+			(effects
+				(font
+					(size 1.27 1.27)
+				)
+			)
+		)
+		(property "Footprint" "SynthStuff:Toggle_Switch_THT"
+			(at 181.61 49.53 0)
+			(effects
+				(font
+					(size 1.27 1.27)
+				)
+				(hide yes)
+			)
+		)
+		(property "Datasheet" "~"
+			(at 181.61 52.07 0)
+			(effects
+				(font
+					(size 1.27 1.27)
+				)
+				(hide yes)
+			)
+		)
+		(property "Description" "Switch, single pole double throw"
+			(at 181.61 59.69 0)
+			(effects
+				(font
+					(size 1.27 1.27)
+				)
+				(hide yes)
+			)
+		)
+		(pin "1"
+		)
+		(pin "2"
+		)
+		(pin "3"
+		)
+		(instances
+			(project ""
+				(path "/58f4306d-5387-4983-bb08-41a2313fd315/ce3fef8b-9f1d-4178-b50b-4a046c030679"
+					(reference "SW4")
+					(unit 1)
+				)

Commit message: Component placement in progress
Parts:
- J50: footprint (none) -> Connector_PinSocket_2.54mm:PinSocket_1x06_P2.54mm_Vertical
Changed lines of the file:
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@@
 			)
 		)
-		(property "Footprint" ""
+		(property "Footprint" "Connector_PinSocket_2.54mm:PinSocket_1x06_P2.54mm_Vertical"
 			(at 127 111.76 0)
 			(effects
